File: opto-counter.kicad_sch (KiCad schematic)
At the start: 13 parts, among them J1 IR-REC, J2 qwiic, J3 UPDI, U1 ATtiny404-SS, U2 TSSP6038

Commit message: Use ATtiny1614-SS as the mCPU
Actually, we're targetting to ATtiny3224, which should be pin
compatible.
Parts:
- removed U1: ATtiny404-SS, Package_SO:SOIC-14_3.9x8.7mm_P1.27mm, symbol MCU_Microchip_ATtiny:ATtiny404-SS
- added U1: ATtiny1614-SS, Package_SO:SOIC-14_3.9x8.7mm_P1.27mm, symbol MCU_Microchip_ATtiny:ATtiny1614-SS
Connections:
- net +3V3: now also U1.1 (VCC)
- net GND: now also U1.14 (GND)
- net SCL: now also U1.12 (PA2)
- net SDA: now also U1.11 (PA1)
- net UPDI: now also U1.10 (~{RESET}/PA0)
- net at J1.1 (Pin_1), U2.4 (OUT): now also U1.2 (PA4)
- net at R2.2: now also U1.3 (PA5)
- net at D1.2 (A): now also U1.4 (PA6)
- net at D2.2 (A): now also U1.5 (PA7)
