File: hw/opto-counter.kicad_pcb (KiCad board)
At the start: 2 copper layers, 27.9 x 27.9 mm, 13 parts, among them J1 IR-REC, J2 qwiic, J3 UPDI, U1 ATtiny1614-SS, U2 TSSP6038

Commit message: Use ATtiny3224 as the mCPU in the schematic
Parts:
- U1: value ATtiny1614-SS -> ATtiny3224-SS
Changed lines of the file:
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@@
     (property "Sheetfile" "opto-counter.kicad_sch")
     (property "Sheetname" "")
-    (property "ki_description" "20MHz, 16kB Flash, 2kB SRAM, 256B EEPROM, SOIC-14")
+    (property "ki_description" "20MHz, 32kB Flash, 3kB SRAM, 256B EEPROM, SOIC-14")
     (property "ki_keywords" "AVR 8bit Microcontroller tinyAVR")
     (attr smd)
@@
         (effects (font (size 1 1) (thickness 0.15)))
     )
-    (fp_text value "ATtiny1614-SS" (at 0 5.28) (layer "F.Fab")
+    (fp_text value "ATtiny3224-SS" (at 0 5.28) (layer "F.Fab")
         (effects (font (size 1 1) (thickness 0.15)))
     )
